File: S4/PayloadSheildV5.1.sch (EAGLE design)
At the start: 20 parts, among them U2 ARDUINOR3

Commit message: ready to print
Parts:
- added R2, R3: 4K7, rcl:R-US_0204/5
- 3.3V: device NASAEPO:LD1117V33 -> TEMP:LD1117V33
Connections:
- removed net SCL: ADXL345.SCL, BMP085.SCL, HIH6310.SCL, MAG3110.SCL, U2.A5/SCL
- new net N$9: ADXL345.SCL, BMP085.SCL, HIH6310.SCL, MAG3110.SCL, R2.2, U2.A5/SCL
- net +3V3: now also R2.1, R3.1
- net SDA: now also R3.2
