File: S4/PayloadSheildV5.brd (EAGLE design)
At the start: 184.2 x 63.5 mm, 20 parts, among them U2 ARDUINOR3

Commit message: ready to print
Connections:
- net N$32: now also LOGIC.TXI2; no longer LOGIC.TI02
Changed lines of the file:
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@@
 <signal name="N$32">
 <contactref element="GPSCON" pad="TX"/>
-<contactref element="LOGIC" pad="TI02"/>
+<contactref element="LOGIC" pad="TXI2"/>
 <wire x1="45.72" y1="14.986" x2="49.022" y2="14.986" width="0.8128" layer="16"/>
 </signal>
